Commit message: 完成

File: velodyne_description/urdf/VLP-16.urdf.xacro (robot description, xacro)
@@ -2,5 +2,5 @@
 <robot xmlns:xacro="http://www.ros.org/wiki/xacro" name="VLP-16">
   <xacro:property name="M_PI" value="3.1415926535897931" />
-  <xacro:macro name="VLP-16" params="*origin parent:=base_link name:=velodyne topic:=/velodyne_points hz:=10 lasers:=16 samples:=1875 collision_range:=0.3 min_range:=0.9 max_range:=130.0 noise:=0.008 min_angle:=-${M_PI} max_angle:=${M_PI} gpu:=false">
+  <xacro:macro name="VLP-16" params="*origin parent:=base_link name:=velodyne topic:=/velodyne_points hz:=10 lasers:=80 samples:=1875 collision_range:=0.3 min_range:=0.9 max_range:=130.0 noise:=0.008 min_angle:=-${M_PI} max_angle:=${M_PI} gpu:=false">
     <joint name="${name}_base_mount_joint" type="fixed">
       <xacro:insert_block name="origin" />

File: velodyne_description/urdf/example.urdf.xacro (robot description, xacro)
@@ -1,6 +1,41 @@
 <?xml version="1.0"?>
-<robot xmlns:xacro="http://www.ros.org/wiki/xacro" name="example">
-  <xacro:arg name="gpu" default="false"/>
-  <xacro:property name="gpu" value="$(arg gpu)" />
+<robot xmlns:xacro="http://www.ros.org/wiki/xacro" name="$(arg LiDARName)">
+  <xacro:arg name="topicName" default="LiDAR_points"/>
+  <xacro:arg name="frameName" default="lidar"/>
+  <xacro:arg name="min_range" default="0.9"/>
+  <xacro:arg name="max_range" default="130.0"/>
+  <xacro:arg name="samples" default="440"/>
+  <xacro:arg name="gaussianNoise" default="0.008"/>
+  <xacro:arg name="hz" default="10"/>
+  <xacro:property name="LiDARName" value="$(arg LiDARName)"/>
+  <xacro:property name="topicName" value="$(arg topicName)" />
+  <xacro:property name="frameName" value="$(arg frameName)" />
+  <xacro:property name="min_range" value="$(arg min_range)" />
+  <xacro:property name="max_range" value="$(arg max_range)" />
+  <xacro:property name="samples" default="$(arg samples)"/>
+  <xacro:property name="hz" value="$(arg hz)" />
+  <xacro:property name="gaussianNoise" value="$(arg gaussianNoise)" />
+  <xacro:include filename="$(find velodyne_description)/urdf/LiDAR-80.xacro"/>
+  <!--                          User configuartion                                          -->
+  <xacro:laserModel
+          parent="base_link"
+          name="${LiDARName}"
+          topic="${topicName}"
+          samples="${samples}"
+          noise="${gaussianNoise}"
+          hz="${hz}"
+          frame="${frameName}" >
+    <origin xyz="0 0 0.4" rpy="0 0 0" />
+  </xacro:laserModel>
+  <gazebo >
+    <plugin name="gazebo_ros_lidar_non_uniform" filename="libgazebo_ros_lidar_non_uniform.so">
+      <topicName>${topicName}</topicName>
+      <frameName>${frameName}</frameName>
+      <min_range>${min_range}</min_range>
+      <max_range>${max_range}</max_range>
+      <gaussianNoise>${gaussianNoise}</gaussianNoise>
+    </plugin>
+  </gazebo>
+  <!--                        User configuartion                                          -->
   <!-- Base Footprint -->
   <link name="base_footprint" />
@@ -30,11 +65,3 @@
     </inertial>
   </link>
-  <xacro:include filename="$(find velodyne_description)/urdf/VLP-16.urdf.xacro"/>
-  <xacro:VLP-16 parent="base_link" name="velodyne" topic="/velodyne_points" hz="10" samples="440" gpu="${gpu}">
-    <origin xyz="0 0 0.4" rpy="0 0 0" />
-  </xacro:VLP-16>
-  <xacro:include filename="$(find velodyne_description)/urdf/HDL-32E.urdf.xacro"/>
-  <xacro:HDL-32E parent="base_link" name="velodyne2" topic="/velodyne_points2" hz="10" samples="220" gpu="${gpu}">
-    <origin xyz="0 0 0.6" rpy="0 0 0" />
-  </xacro:HDL-32E>
 </robot>

Commit message: fix frame

File: velodyne_description/urdf/VLP-16.urdf.xacro (robot description, xacro)
@@ -2,5 +2,5 @@
 <robot xmlns:xacro="http://www.ros.org/wiki/xacro" name="VLP-16">
   <xacro:property name="M_PI" value="3.1415926535897931" />
-  <xacro:macro name="VLP-16" params="*origin parent:=base_link name:=velodyne topic:=/velodyne_points hz:=10 lasers:=80 samples:=1875 collision_range:=0.3 min_range:=0.9 max_range:=130.0 noise:=0.008 min_angle:=-${M_PI} max_angle:=${M_PI} gpu:=false">
+  <xacro:macro name="VLP-16" params="*origin parent:=base_link name:=velodyne topic:=/velodyne_points hz:=10 lasers:=16 samples:=1875 collision_range:=0.3 min_range:=0.9 max_range:=130.0 noise:=0.008 min_angle:=-${M_PI} max_angle:=${M_PI} gpu:=false">
     <joint name="${name}_base_mount_joint" type="fixed">
       <xacro:insert_block name="origin" />

File: velodyne_description/urdf/example.urdf.xacro (robot description, xacro)
@@ -1,67 +1,54 @@
 <?xml version="1.0"?>
-<robot xmlns:xacro="http://www.ros.org/wiki/xacro" name="$(arg LiDARName)">
-  <xacro:arg name="topicName" default="LiDAR_points"/>
-  <xacro:arg name="frameName" default="lidar"/>
-  <xacro:arg name="min_range" default="0.9"/>
-  <xacro:arg name="max_range" default="130.0"/>
-  <xacro:arg name="samples" default="440"/>
-  <xacro:arg name="gaussianNoise" default="0.008"/>
-  <xacro:arg name="hz" default="10"/>
-  <xacro:property name="LiDARName" value="$(arg LiDARName)"/>
-  <xacro:property name="topicName" value="$(arg topicName)" />
-  <xacro:property name="frameName" value="$(arg frameName)" />
-  <xacro:property name="min_range" value="$(arg min_range)" />
-  <xacro:property name="max_range" value="$(arg max_range)" />
-  <xacro:property name="samples" default="$(arg samples)"/>
-  <xacro:property name="hz" value="$(arg hz)" />
-  <xacro:property name="gaussianNoise" value="$(arg gaussianNoise)" />
-  <xacro:include filename="$(find velodyne_description)/urdf/LiDAR-80.xacro"/>
+<robot xmlns:xacro="http://www.ros.org/wiki/xacro" name="robot">
+  <xacro:include filename="$(find velodyne_description)/urdf/RS-Ruby80.urdf.xacro"/>
+  <xacro:include filename="$(find velodyne_description)/urdf/VLP-16.urdf.xacro"/>
   <!--                          User configuartion                                          -->
-  <xacro:laserModel
+  <xacro:RS-Ruby80
           parent="base_link"
-          name="${LiDARName}"
-          topic="${topicName}"
-          samples="${samples}"
-          noise="${gaussianNoise}"
-          hz="${hz}"
-          frame="${frameName}" >
-    <origin xyz="0 0 0.4" rpy="0 0 0" />
-  </xacro:laserModel>
-  <gazebo >
-    <plugin name="gazebo_ros_lidar_non_uniform" filename="libgazebo_ros_lidar_non_uniform.so">
-      <topicName>${topicName}</topicName>
-      <frameName>${frameName}</frameName>
-      <min_range>${min_range}</min_range>
-      <max_range>${max_range}</max_range>
-      <gaussianNoise>${gaussianNoise}</gaussianNoise>
-    </plugin>
-  </gazebo>
+          name="Ruby80"
+          topic="Ruby80"
+          samples="1800"
+          noise="0.008"
+          frame="Ruby80frame"
+          gpu="true">
+    <origin xyz="0 0 0" rpy="0 0 0" />
+  </xacro:RS-Ruby80>
   <!--                        User configuartion                                          -->
-  <!-- Base Footprint -->
-  <link name="base_footprint" />
+<!--  &lt;!&ndash; Base Footprint &ndash;&gt;-->
+  <link name="base_footprint"/>
   <!-- Base Link -->
   <joint name="footprint" type="fixed" >
-   <parent link="base_footprint" />
+    <parent link="base_footprint" />
     <child link="base_link" />
-    <origin xyz="0 0 0.05" rpy="0 0 0" />
+    <origin xyz="0 0 0" rpy="0 0 0" />
   </joint>
   <link name="base_link" >
+    <inertial>
+      <origin
+              xyz="0.10076 -0.52187 5.5716E-07"
+              rpy="0 0 0" />
+      <mass
+              value="0.2" />
+      <inertia
+              ixx="1e-10"
+              ixy="1e-10"
+              ixz="1e-10"
+              iyy="1e-10"
+              iyz="1e-10"
+              izz="1e-10" />
+    </inertial>
     <visual>
       <geometry>
-        <box size="0.5 0.5 0.1" />
+        <box size="0.1 0.1 0.01" />
       </geometry>
     </visual>
     <collision>
+      <origin
+              xyz="0 0 0"
+              rpy="0 0 0" />
       <geometry>
-        <box size="0.5 0.5 0.1" />
+        <box size="0.1 0.1 0.01" />
       </geometry>
     </collision>
-    <inertial>
-      <origin xyz="0 0 0"/>
-      <mass value="10"/>
-      <inertia ixx="3.0" ixy="0.0" ixz="0.0"
-               iyy="3.0" iyz="0.0"
-               izz="3.0" />
-    </inertial>
   </link>
 </robot>
