Commit message: 修改多机bug

File: velodyne_description/urdf/RS-Ruby80.urdf.xacro (robot description, xacro)
@@ -54,12 +54,12 @@
   min_range:=1    max_range:=230.0
   ">
-    <joint name="${parent}_${frame}_fixed_joint"  type="revolute">
+    <joint name="${ns}_${parent}_${frame}_fixed_joint"  type="revolute">
       <xacro:insert_block name="origin" />
       <parent link="${parent}" />
-      <child link="${frame}" />
+      <child link="${ns}_${frame}" />
       <axis xyz="0 0 1"/>
       <limit  lower="-1e-5" upper="1e-5" effort="1e-5" velocity="1e-5" />
     </joint>
-    <link name="${frame}">
+    <link name="${ns}_${frame}">
       <inertial>
         <mass value="3.75"/>
@@ -92,5 +92,5 @@
       <plugin name="${lib}" filename="lib${lib}.so">
         <topicName>${topic}</topicName>
-        <frameName>${frame}</frameName>
+        <frameName>${ns}_${frame}</frameName>
         <namespace>${ns}</namespace>
         <min_range>${min_range}</min_range>
@@ -98,5 +98,5 @@
       </plugin>
     </gazebo>
-    <gazebo reference="${frame}">
+    <gazebo reference="${ns}_${frame}">
       <xacro:LiDARSensorGen name="sensor-sector" suffix="1"
                             visualize="${visualize}" hz="${hz}" gpu="${gpu}" noise="0.008"

File: velodyne_description/urdf/example.urdf.xacro (robot description, xacro)
@@ -5,11 +5,12 @@
   <!--                          User configuartion                                          -->
   <xacro:RS-Ruby80
-          parent="base_link"
+          parent="top_link"
           name="Ruby80"
           topic="Ruby80"
-          samples="1800"
+          samples="180"
           noise="0.008"
-          frame="Ruby80frame"
-          gpu="true">
+          frame="Ruby80"
+          gpu="false"
+          ns="$(arg robot_namespace)">
     <origin xyz="0 0 0" rpy="0 0 0" />
   </xacro:RS-Ruby80>
@@ -26,5 +27,39 @@
     <inertial>
       <origin
-              xyz="0.10076 -0.52187 5.5716E-07"
+              xyz="0 0 0"
+              rpy="0 0 0" />
+      <mass
+              value="200" />
+      <inertia
+              ixx="1e-10"
+              ixy="1e-10"
+              ixz="1e-10"
+              iyy="1e-10"
+              iyz="1e-10"
+              izz="1e-10" />
+    </inertial>
+    <visual>
+      <geometry>
+        <box size="0.1 0.1 0.01" />
+      </geometry>
+    </visual>
+    <collision>
+      <origin
+              xyz="0 0 0"
+              rpy="0 0 0" />
+      <geometry>
+        <box size="0.1 0.1 0.01" />
+      </geometry>
+    </collision>
+  </link>
+  <joint name="mount_joint" type="fixed" >
+    <parent link="base_link" />
+    <child link="top_link" />
+    <origin xyz="0 0 0.4" rpy="0 0 0" />
+  </joint>
+  <link name="top_link" >
+    <inertial>
+      <origin
+              xyz="0 0 0.4"
               rpy="0 0 0" />
       <mass

Commit message: 修复lidar在多机下tf的bug

File: velodyne_description/urdf/RS-Ruby80.urdf.xacro (robot description, xacro)
@@ -64,5 +64,5 @@
       <inertial>
         <mass value="3.75"/>
-        <origin xyz="-0.0443 0 0.00625" rpy="0 0 0"/>
+        <origin xyz="0 0 0" rpy="0 0 0"/>
         <inertia ixx="${(1.0 * (3.0*0.04267*0.04267 + 0.14424*0.14424)) / 12.0}" ixy="0" ixz="0"
                  iyy="${(1.0 * (3.0*0.04267*0.04267 + 0.14424*0.14424)) / 12.0}" iyz="0"
@@ -70,5 +70,5 @@
       </inertial>
       <visual>
-        <origin xyz="-0.0443 0 0.00625" rpy="0 0 0"/>
+        <origin xyz="0 0 0" rpy="0 0 0"/>
         <geometry>
           <mesh filename="package://velodyne_description/meshes/RS_Ruby80.STL" />
@@ -76,5 +76,5 @@
       </visual>
       <collision>
-        <origin xyz="-0.0443 0 0.00625" rpy="0 0 0"/>
+        <origin xyz="0 0 0" rpy="0 0 0"/>
         <geometry>
           <mesh filename="package://velodyne_description/meshes/RS_Ruby80.STL" />

File: velodyne_description/urdf/example.urdf.xacro (robot description, xacro)
@@ -1,89 +1,89 @@
 <?xml version="1.0"?>
 <robot xmlns:xacro="http://www.ros.org/wiki/xacro" name="robot">
-  <xacro:include filename="$(find velodyne_description)/urdf/RS-Ruby80.urdf.xacro"/>
-  <xacro:include filename="$(find velodyne_description)/urdf/VLP-16.urdf.xacro"/>
-  <!--                          User configuartion                                          -->
-  <xacro:RS-Ruby80
-          parent="top_link"
-          name="Ruby80"
-          topic="Ruby80"
-          samples="180"
-          noise="0.008"
-          frame="Ruby80"
-          gpu="false"
-          ns="$(arg robot_namespace)">
-    <origin xyz="0 0 0" rpy="0 0 0" />
-  </xacro:RS-Ruby80>
-  <!--                        User configuartion                                          -->
-<!--  &lt;!&ndash; Base Footprint &ndash;&gt;-->
-  <link name="base_footprint"/>
-  <!-- Base Link -->
-  <joint name="footprint" type="fixed" >
-    <parent link="base_footprint" />
-    <child link="base_link" />
-    <origin xyz="0 0 0" rpy="0 0 0" />
-  </joint>
-  <link name="base_link" >
-    <inertial>
-      <origin
-              xyz="0 0 0"
-              rpy="0 0 0" />
-      <mass
-              value="200" />
-      <inertia
-              ixx="1e-10"
-              ixy="1e-10"
-              ixz="1e-10"
-              iyy="1e-10"
-              iyz="1e-10"
-              izz="1e-10" />
-    </inertial>
-    <visual>
-      <geometry>
-        <box size="0.1 0.1 0.01" />
-      </geometry>
-    </visual>
-    <collision>
-      <origin
-              xyz="0 0 0"
-              rpy="0 0 0" />
-      <geometry>
-        <box size="0.1 0.1 0.01" />
-      </geometry>
-    </collision>
-  </link>
-  <joint name="mount_joint" type="fixed" >
-    <parent link="base_link" />
-    <child link="top_link" />
-    <origin xyz="0 0 0.4" rpy="0 0 0" />
-  </joint>
-  <link name="top_link" >
-    <inertial>
-      <origin
-              xyz="0 0 0.4"
-              rpy="0 0 0" />
-      <mass
-              value="0.2" />
-      <inertia
-              ixx="1e-10"
-              ixy="1e-10"
-              ixz="1e-10"
-              iyy="1e-10"
-              iyz="1e-10"
-              izz="1e-10" />
-    </inertial>
-    <visual>
-      <geometry>
-        <box size="0.1 0.1 0.01" />
-      </geometry>
-    </visual>
-    <collision>
-      <origin
-              xyz="0 0 0"
-              rpy="0 0 0" />
-      <geometry>
-        <box size="0.1 0.1 0.01" />
-      </geometry>
-    </collision>
-  </link>
+    <xacro:include filename="$(find velodyne_description)/urdf/RS-Ruby80.urdf.xacro"/>
+    <xacro:include filename="$(find velodyne_description)/urdf/VLP-16.urdf.xacro"/>
+    <!--                          User configuartion                                          -->
+    <xacro:RS-Ruby80
+            parent="top_link"
+            name="Ruby80"
+            topic="Ruby80"
+            samples="3600"
+            noise="0.008"
+            frame="Ruby80"
+            gpu="true"
+            ns="$(arg robot_namespace)">
+        <origin xyz="0 0 0" rpy="0 0 0"/>
+    </xacro:RS-Ruby80>
+    <!--                        User configuartion                                          -->
+    <!--  &lt;!&ndash; Base Footprint &ndash;&gt;-->
+    <link name="base_footprint"/>
+    <!-- Base Link -->
+    <joint name="footprint" type="fixed">
+        <parent link="base_footprint"/>
+        <child link="base_link"/>
+        <origin xyz="0 0 0" rpy="0 0 0"/>
+    </joint>
+    <link name="base_link">
+        <inertial>
+            <origin
+                    xyz="0 0 0"
+                    rpy="0 0 0"/>
+            <mass
+                    value="200"/>
+            <inertia
+                    ixx="1e-10"
+                    ixy="1e-10"
+                    ixz="1e-10"
+                    iyy="1e-10"
+                    iyz="1e-10"
+                    izz="1e-10"/>
+        </inertial>
+        <visual>
+            <geometry>
+                <box size="0.1 0.1 0.01"/>
+            </geometry>
+        </visual>
+        <collision>
+            <origin
+                    xyz="0 0 0"
+                    rpy="0 0 0"/>
+            <geometry>
+                <box size="0.1 0.1 0.01"/>
+            </geometry>
+        </collision>
+    </link>
+    <joint name="mount_joint" type="fixed">
+        <parent link="base_link"/>
+        <child link="top_link"/>
+        <origin xyz="0 0 0.4" rpy="0 0 0"/>
+    </joint>
+    <link name="top_link">
+        <inertial>
+            <origin
+                    xyz="0 0 0.4"
+                    rpy="0 0 0"/>
+            <mass
+                    value="0.2"/>
+            <inertia
+                    ixx="1e-10"
+                    ixy="1e-10"
+                    ixz="1e-10"
+                    iyy="1e-10"
+                    iyz="1e-10"
+                    izz="1e-10"/>
+        </inertial>
+        <visual>
+            <geometry>
+                <box size="0.1 0.1 0.01"/>
+            </geometry>
+        </visual>
+        <collision>
+            <origin
+                    xyz="0 0 0"
+                    rpy="0 0 0"/>
+            <geometry>
+                <box size="0.1 0.1 0.01"/>
+            </geometry>
+        </collision>
+    </link>
 </robot>

Commit message: 完成默认功能标注工具

File: velodyne_description/urdf/RS-Ruby80.urdf.xacro (robot description, xacro)
@@ -1,6 +1,6 @@
 <?xml version="1.0"?>
 <robot xmlns:xacro="http://www.ros.org/wiki/xacro" name="LiDAR-80">
-  <xacro:property name="M_PI" value="3.1415926535897931" />
-  <xacro:macro name="LiDARSensorGen" params="
+    <xacro:property name="M_PI" value="3.1415926535897931"/>
+    <xacro:macro name="LiDARSensorGen" params="
   name      suffix
   visualize:=false      gpu:=false      hz:=10
@@ -10,110 +10,115 @@
   v_min_angle:=-${M_PI/12}         v_max_angle:=${15*M_PI/12}
   ">
-    <xacro:if value="${gpu}">
-      <xacro:property name="type" value="gpu_ray"/>
-    </xacro:if>
-    <xacro:unless value="${gpu}">
-      <xacro:property name="type" value="ray"/>
-    </xacro:unless>
-    <sensor type="${type}" name="${name}-${suffix}">
-      <visualize>${visualize}</visualize>
-      <update_rate>${hz}</update_rate>
-      <ray>
-        <scan>
-          <horizontal>
-            <samples>${samples}</samples>
-            <resolution>1</resolution>
-            <min_angle>${min_angle}</min_angle>
-            <max_angle>${max_angle}</max_angle>
-          </horizontal>
-          <vertical>
-            <samples>${lasers}</samples>
-            <resolution>1</resolution>
-            <min_angle>${v_min_angle}</min_angle>
-            <max_angle>${v_max_angle}</max_angle>
-          </vertical>
-        </scan>
-        <range>
-          <min>${min_range}</min>
-          <max>${max_range}</max>
-          <resolution>0.001</resolution>
-        </range>
-        <noise>
-          <type>gaussian</type>
-          <mean>0.0</mean>
-          <stddev>${noise}</stddev>
-        </noise>
-      </ray>
-    </sensor>
-  </xacro:macro>
-  <xacro:macro name="RS-Ruby80"  params="
+        <xacro:if value="${gpu}">
+            <xacro:property name="type" value="gpu_ray"/>
+        </xacro:if>
+        <xacro:unless value="${gpu}">
+            <xacro:property name="type" value="ray"/>
+        </xacro:unless>
+        <sensor type="${type}" name="${name}-${suffix}">
+            <visualize>${visualize}</visualize>
+            <update_rate>${hz}</update_rate>
+            <ray>
+                <scan>
+                    <horizontal>
+                        <samples>${samples}</samples>
+                        <resolution>1</resolution>
+                        <min_angle>${min_angle}</min_angle>
+                        <max_angle>${max_angle}</max_angle>
+                    </horizontal>
+                    <vertical>
+                        <samples>${lasers}</samples>
+                        <resolution>1</resolution>
+                        <min_angle>${v_min_angle}</min_angle>
+                        <max_angle>${v_max_angle}</max_angle>
+                    </vertical>
+                </scan>
+                <range>
+                    <min>${min_range}</min>
+                    <max>${max_range}</max>
+                    <resolution>0.001</resolution>
+                </range>
+                <noise>
+                    <type>gaussian</type>
+                    <mean>0.0</mean>
+                    <stddev>${noise}</stddev>
+                </noise>
+            </ray>
+        </sensor>
+    </xacro:macro>
+    <xacro:macro name="RS-Ruby80" params="
   name      parent      *origin
-  frame      topic      ns:=''
+  frame      topic      ns:=false
   visualize:=false      gpu:=false      hz:=10
   samples:=1800      noise:=0.008
   min_range:=1    max_range:=230.0
   ">
-    <joint name="${ns}_${parent}_${frame}_fixed_joint"  type="revolute">
-      <xacro:insert_block name="origin" />
-      <parent link="${parent}" />
-      <child link="${ns}_${frame}" />
-      <axis xyz="0 0 1"/>
-      <limit  lower="-1e-5" upper="1e-5" effort="1e-5" velocity="1e-5" />
-    </joint>
-    <link name="${ns}_${frame}">
-      <inertial>
-        <mass value="3.75"/>
-        <origin xyz="0 0 0" rpy="0 0 0"/>
-        <inertia ixx="${(1.0 * (3.0*0.04267*0.04267 + 0.14424*0.14424)) / 12.0}" ixy="0" ixz="0"
-                 iyy="${(1.0 * (3.0*0.04267*0.04267 + 0.14424*0.14424)) / 12.0}" iyz="0"
-                 izz="${0.5 * 1.0 * (0.04267*0.04267)}"/>
-      </inertial>
-      <visual>
-        <origin xyz="0 0 0" rpy="0 0 0"/>
-        <geometry>
-          <mesh filename="package://velodyne_description/meshes/RS_Ruby80.STL" />
-        </geometry>
-      </visual>
-      <collision>
-        <origin xyz="0 0 0" rpy="0 0 0"/>
-        <geometry>
-          <mesh filename="package://velodyne_description/meshes/RS_Ruby80.STL" />
-        </geometry>
-      </collision>
-    </link>
-    <xacro:if value="${gpu}">
-      <xacro:property name="lib" value="gazebo_ros_custom_gpu_lidar"/>
-    </xacro:if>
-    <xacro:unless value="${gpu}">
-      <xacro:property name="lib" value="gazebo_ros_custom_lidar"/>
-    </xacro:unless>
-    <!-- Custom LiDAR Config -->
-    <gazebo >
-      <plugin name="${lib}" filename="lib${lib}.so">
-        <topicName>${topic}</topicName>
-        <frameName>${ns}_${frame}</frameName>
-        <namespace>${ns}</namespace>
-        <min_range>${min_range}</min_range>
-        <max_range>${max_range}</max_range>
-      </plugin>
-    </gazebo>
-    <gazebo reference="${ns}_${frame}">
-      <xacro:LiDARSensorGen name="sensor-sector" suffix="1"
-                            visualize="${visualize}" hz="${hz}" gpu="${gpu}" noise="0.008"
-                            samples="${samples}" lasers="15     +1"
-                            v_max_angle="${15         *M_PI/180.0}"
-                            v_min_angle="${1.91       *M_PI/180.0}"/>
-      <xacro:LiDARSensorGen name="sensor-sector" suffix="2"
-                            visualize="${visualize}" hz="${hz}" gpu="${gpu}" noise="0.008"
-                            samples="${samples}" lasers="40     -2"
-                            v_max_angle="${1.01       *M_PI/180.0}"
-                            v_min_angle="${-2.99      *M_PI/180.0}"/>
-      <xacro:LiDARSensorGen name="sensor-sector" suffix="3"
-                            visualize="${visualize}" hz="${hz}" gpu="${gpu}" noise="0.008"
-                            samples="${samples}" lasers="25     +1"
-                            v_max_angle="${-3.89      *M_PI/180.0}"
-                            v_min_angle="${-25        *M_PI/180.0}"/>
-    </gazebo>
-    <!-- Custom LiDAR Config -->
-  </xacro:macro>
+        <joint name="${parent}_${frame}_fixed_joint" type="revolute">
+            <xacro:insert_block name="origin"/>
+            <parent link="${parent}"/>
+            <child link="${frame}"/>
+            <axis xyz="0 0 1"/>
+            <limit lower="-1e-5" upper="1e-5" effort="1e-5" velocity="1e-5"/>
+        </joint>
+        <link name="${frame}">
+            <inertial>
+                <mass value="3.75"/>
+                <origin xyz="0 0 0" rpy="0 0 0"/>
+                <inertia ixx="${(1.0 * (3.0*0.04267*0.04267 + 0.14424*0.14424)) / 12.0}" ixy="0" ixz="0"
+                         iyy="${(1.0 * (3.0*0.04267*0.04267 + 0.14424*0.14424)) / 12.0}" iyz="0"
+                         izz="${0.5 * 1.0 * (0.04267*0.04267)}"/>
+            </inertial>
+            <visual>
+                <origin xyz="0 0 0" rpy="0 0 0"/>
+                <geometry>
+                    <mesh filename="package://velodyne_description/meshes/RS_Ruby80.STL"/>
+                </geometry>
+            </visual>
+            <collision>
+                <origin xyz="0 0 0" rpy="0 0 0"/>
+                <geometry>
+                    <mesh filename="package://velodyne_description/meshes/RS_Ruby80.STL"/>
+                </geometry>
+            </collision>
+        </link>
+        <xacro:if value="${gpu}">
+            <xacro:property name="lib" value="gazebo_ros_custom_gpu_lidar"/>
+        </xacro:if>
+        <xacro:unless value="${gpu}">
+            <xacro:property name="lib" value="gazebo_ros_custom_lidar"/>
+        </xacro:unless>
+        <!-- Custom LiDAR Config -->
+        <gazebo>
+            <plugin name="${lib}" filename="lib${lib}.so">
+                <topicName>${topic}</topicName>
+                <frameName>${frame}</frameName>
+                <xacro:if value="${ns=='false'}">
+                    <namespace>/</namespace>
+                </xacro:if>
+                <xacro:unless value="${ns=='false'}">
+                    <namespace>${ns}</namespace>
+                </xacro:unless>
+                <min_range>${min_range}</min_range>
+                <max_range>${max_range}</max_range>
+            </plugin>
+        </gazebo>
+        <gazebo reference="${frame}">
+            <xacro:LiDARSensorGen name="sensor-sector" suffix="1"
+                                  visualize="${visualize}" hz="${hz}" gpu="${gpu}" noise="0.008"
+                                  samples="${samples}" lasers="15     +1"
+                                  v_max_angle="${15         *M_PI/180.0}"
+                                  v_min_angle="${1.91       *M_PI/180.0}"/>
+            <xacro:LiDARSensorGen name="sensor-sector" suffix="2"
+                                  visualize="${visualize}" hz="${hz}" gpu="${gpu}" noise="0.008"
+                                  samples="${samples}" lasers="40     -2"
+                                  v_max_angle="${1.01       *M_PI/180.0}"
+                                  v_min_angle="${-2.99      *M_PI/180.0}"/>
+            <xacro:LiDARSensorGen name="sensor-sector" suffix="3"
+                                  visualize="${visualize}" hz="${hz}" gpu="${gpu}" noise="0.008"
+                                  samples="${samples}" lasers="25     +1"
+                                  v_max_angle="${-3.89      *M_PI/180.0}"
+                                  v_min_angle="${-25        *M_PI/180.0}"/>
+        </gazebo>
+        <!-- Custom LiDAR Config -->
+    </xacro:macro>
 </robot>

Commit message: 使用新方法构建非均匀线束LiDAR

File: velodyne_description/urdf/RS-Ruby80.urdf.xacro (robot description, xacro)
@@ -57,9 +57,9 @@
             <xacro:insert_block name="origin"/>
             <parent link="${parent}"/>
-            <child link="${frame}"/>
+            <child link="${ns}/${frame}"/>
             <axis xyz="0 0 1"/>
             <limit lower="-1e-5" upper="1e-5" effort="1e-5" velocity="1e-5"/>
         </joint>
-        <link name="${frame}">
+        <link name="${ns}/${frame}">
             <inertial>
                 <mass value="3.75"/>

File: velodyne_description/urdf/VLP-16.urdf.xacro (robot description, xacro)
@@ -2,5 +2,5 @@
 <robot xmlns:xacro="http://www.ros.org/wiki/xacro" name="VLP-16">
   <xacro:property name="M_PI" value="3.1415926535897931" />
-  <xacro:macro name="VLP-16" params="*origin parent:=base_link name:=velodyne topic:=/velodyne_points hz:=10 lasers:=16 samples:=1875 collision_range:=0.3 min_range:=0.9 max_range:=130.0 noise:=0.008 min_angle:=-${M_PI} max_angle:=${M_PI} gpu:=false">
+  <xacro:macro name="VLP-16" params="*origin  parent:=base_link name:=velodyne topic:=/velodyne_points hz:=10 lasers:=16 samples:=1875 collision_range:=0.3 min_range:=0.9 max_range:=130.0 noise:=0.008 min_angle:=-${M_PI} max_angle:=${M_PI} gpu:=false">
     <joint name="${name}_base_mount_joint" type="fixed">
       <xacro:insert_block name="origin" />
@@ -125,4 +125,5 @@
           </ray>
           <plugin name="gazebo_ros_laser_controller" filename="libgazebo_ros_velodyne_laser.so">
+            <namespace>excavator</namespace>
             <topicName>${topic}</topicName>
             <frameName>${name}</frameName>

File: velodyne_description/urdf/example.urdf.xacro (robot description, xacro)
@@ -1,18 +1,16 @@
 <?xml version="1.0"?>
 <robot xmlns:xacro="http://www.ros.org/wiki/xacro" name="robot">
+    <xacro:include filename="$(find velodyne_description)/urdf/Customized.urdf.xacro"/>
     <xacro:include filename="$(find velodyne_description)/urdf/RS-Ruby80.urdf.xacro"/>
     <xacro:include filename="$(find velodyne_description)/urdf/VLP-16.urdf.xacro"/>
     <!--                          User configuartion                                          -->
-    <xacro:RS-Ruby80
-            parent="top_link"
+    <xacro:Customized_LiDAR
             name="Ruby80"
             topic="Ruby80"
-            samples="3600"
-            noise="0.008"
-            frame="Ruby80"
             gpu="true"
-            ns="$(arg robot_namespace)">
+            ns="$(arg robot_namespace)"
+            parent="top_link">
         <origin xyz="0 0 0" rpy="0 0 0"/>
-    </xacro:RS-Ruby80>
+    </xacro:Customized_LiDAR>
     <!--                        User configuartion                                          -->
     <!--  &lt;!&ndash; Base Footprint &ndash;&gt;-->
